File: Hardware/PCB.kicad_pcb (KiCad board)
At the start: 2 copper layers, 53.4 x 22 mm, 9 parts, among them J1 Conn_01x04_Pin, U1 ME54BS01_V1.0, U2 MCP1700x-330xxTO

Commit message: Update PCB with new pin outs
Connections:
- U1 pad 12: /p1reading -> unconnected-(U1-P1.04/AIN0-Pad12)
- U1 pad 21: unconnected-(U1-P2.09-Pad21) -> /reset
- U1 pad 22: unconnected-(U1-P2.10-Pad22) -> /indicator
- U1 pad 24: /reset -> unconnected-(U1-P0.01-Pad24)
- U1 pad 4: unconnected-(U1-P1.11/AIN4-Pad4) -> /p2reading
- U1 pad 5: unconnected-(U1-P1.12/AIN5-Pad5) -> /p1reading
- U1 pad 9: /p2reading -> unconnected-(U1-P1.05/AIN1-Pad9)
Routing:
- net /p1reading: track 25.4 -> 33.1 mm
- net /p2reading: track 21.1 -> 26.5 mm
- net /reset: track 47.4 -> 44.2 mm
- net unconnected-(U1-P1.05/AIN1-Pad9): track 0.00 -> 0.50 mm
- net unconnected-(U1-P1.04/AIN0-Pad12): track 0.00 -> 0.50 mm

Commit message: Update the PCB
Parts:
- added D1: LED, LED_SMD:LED_0805_2012Metric, F.Cu at (52.7, 71.2)
- added R4: R, Resistor_SMD:R_0805_2012Metric, F.Cu at (57.4, 71.2)
Routing:
- net /indicator: track 0.00 -> 29.8 mm
- net Net-(D1-A): track 0.00 -> 2.84 mm
- net GND: track 7.87 -> 9.52 mm, vias 2 -> 3
